Commit message: temp commit

File: cartographer_ros/urdf/safmc_2d.urdf (robot description, URDF)
Before this commit: robot cartographer_backpack_2d, 2 links, 1 joints
Links:
- added link imu_link; visual box size=0.00 0.00 0.00
Joints:
- added joint imu_link_joint: type fixed, parent base_link, child imu_link, origin xyz=0 0 0 rpy=0 0 0
- joint rplidar_link_joint: origin xyz=0 0 0 rpy=0 0 1.57008 -> xyz=0 0 0 rpy=0 0 1.57
